Commit message: Split-urdf now aligns base joint 0 with world z and can be invoked as a standalone simulator with split_urdf_draft::simulate.

File: src/robot/urdf/axol-left.urdf (robot description, URDF)
Before this commit: robot assembly, 20 links, 19 joints
Joints:
- joint __split_left_arm_base_to_original_root: origin xyz=-0.13000000000000095 0 -0.85999999999999999 rpy=0 0 -1.5707963267948966 -> xyz=-0.85999999999999999 0 0.13000000000000095 rpy=-1.5707963267948977 0 -1.5707963267948966

File: src/robot/urdf/axol-right.urdf (robot description, URDF)
Before this commit: robot assembly, 20 links, 19 joints
Joints:
- joint __split_right_arm_base_to_original_root: origin xyz=0.12999999999999975 0 -0.85999999999999999 rpy=0 0 -1.5707963267948966 -> xyz=0.85999999999999999 0 0.12999999999999975 rpy=1.5707963267948963 0 -1.5707963267948966

Commit message: cleaned up comments. Ready to send to Almond alongside a blank robot-interface: note that while rudimentary tests have been performed in simulation nothing has been run on hardware and the implementation is likely over-complex.

File: src/robot/urdf/axol-left.urdf (robot description, URDF)
Before this commit: robot assembly, 20 links, 19 joints
Links:
- link base: geometry collision mesh filename=meshes/Base.stl scale=1 1 1; visual mesh filename=meshes/Base.stl scale=1 1 1
- link left_e1: geometry collision mesh filename=meshes/Left_E1.stl scale=1 1 1; visual mesh filename=meshes/Left_E1.stl scale=1 1 1
- link left_e2: geometry collision mesh filename=meshes/Left_E2.stl scale=1 1 1; visual mesh filename=meshes/Left_E2.stl scale=1 1 1
- link left_gripper: geometry collision mesh filename=meshes/Left_Gripper.stl scale=1 1 1; visual mesh filename=meshes/Left_Gripper.stl scale=1 1 1
- link left_s2: geometry collision mesh filename=meshes/Left_S2.stl scale=1 1 1; visual mesh filename=meshes/Left_S2.stl scale=1 1 1
- link left_s3: geometry collision mesh filename=meshes/Left_S3.stl scale=1 1 1; visual mesh filename=meshes/Left_S3.stl scale=1 1 1
- link left_w0: geometry collision mesh filename=meshes/Left_W0.stl scale=1 1 1; visual mesh filename=meshes/Left_W0.stl scale=1 1 1
- link left_w1: geometry collision mesh filename=meshes/Left_W1.stl scale=1 1 1; visual mesh filename=meshes/Left_W1.stl scale=1 1 1
- link left_w2: geometry collision mesh filename=meshes/Left_W2.stl scale=1 1 1; visual mesh filename=meshes/Left_W2.stl scale=1 1 1
- link right_e1: geometry collision mesh filename=meshes/Right_E1.stl scale=1 1 1; visual mesh filename=meshes/Right_E1.stl scale=1 1 1
- link right_e2: geometry collision mesh filename=meshes/Right_E2.stl scale=1 1 1; visual mesh filename=meshes/Right_E2.stl scale=1 1 1
- link right_gripper: geometry collision mesh filename=meshes/Right_Gripper.stl scale=1 1 1; visual mesh filename=meshes/Right_Gripper.stl scale=1 1 1
- link right_s2: geometry collision mesh filename=meshes/Right_S2.stl scale=1 1 1; visual mesh filename=meshes/Right_S2.stl scale=1 1 1
- link right_s3: geometry collision mesh filename=meshes/Right_S3.stl scale=1 1 1; visual mesh filename=meshes/Right_S3.stl scale=1 1 1
- link right_w0: geometry collision mesh filename=meshes/Right_W0.stl scale=1 1 1; visual mesh filename=meshes/Right_W0.stl scale=1 1 1
- link right_w1: geometry collision mesh filename=meshes/Right_W1.stl scale=1 1 1; visual mesh filename=meshes/Right_W1.stl scale=1 1 1
- link right_w2: geometry collision mesh filename=meshes/Right_W2.stl scale=1 1 1; visual mesh filename=meshes/Right_W2.stl scale=1 1 1
- link s1: geometry collision mesh filename=meshes/S1.stl scale=1 1 1; visual mesh filename=meshes/S1.stl scale=1 1 1
Joints:
- joint __split_left_arm_base_to_original_root: origin xyz=-0.85999999999999999 0 0.13000000000000095 rpy=-1.5707963267948977 0 -1.5707963267948966 -> xyz=0.85999999999999999 0 -0.13000000000000095 rpy=1.5707963267948954 0 -1.5707963267948966

File: src/robot/urdf/axol-right.urdf (robot description, URDF)
Before this commit: robot assembly, 20 links, 19 joints
Links:
- link base: geometry collision mesh filename=meshes/Base.stl scale=1 1 1; visual mesh filename=meshes/Base.stl scale=1 1 1
- link left_e1: geometry collision mesh filename=meshes/Left_E1.stl scale=1 1 1; visual mesh filename=meshes/Left_E1.stl scale=1 1 1
- link left_e2: geometry collision mesh filename=meshes/Left_E2.stl scale=1 1 1; visual mesh filename=meshes/Left_E2.stl scale=1 1 1
- link left_gripper: geometry collision mesh filename=meshes/Left_Gripper.stl scale=1 1 1; visual mesh filename=meshes/Left_Gripper.stl scale=1 1 1
- link left_s2: geometry collision mesh filename=meshes/Left_S2.stl scale=1 1 1; visual mesh filename=meshes/Left_S2.stl scale=1 1 1
- link left_s3: geometry collision mesh filename=meshes/Left_S3.stl scale=1 1 1; visual mesh filename=meshes/Left_S3.stl scale=1 1 1
- link left_w0: geometry collision mesh filename=meshes/Left_W0.stl scale=1 1 1; visual mesh filename=meshes/Left_W0.stl scale=1 1 1
- link left_w1: geometry collision mesh filename=meshes/Left_W1.stl scale=1 1 1; visual mesh filename=meshes/Left_W1.stl scale=1 1 1
- link left_w2: geometry collision mesh filename=meshes/Left_W2.stl scale=1 1 1; visual mesh filename=meshes/Left_W2.stl scale=1 1 1
- link right_e1: geometry collision mesh filename=meshes/Right_E1.stl scale=1 1 1; visual mesh filename=meshes/Right_E1.stl scale=1 1 1
- link right_e2: geometry collision mesh filename=meshes/Right_E2.stl scale=1 1 1; visual mesh filename=meshes/Right_E2.stl scale=1 1 1
- link right_gripper: geometry collision mesh filename=meshes/Right_Gripper.stl scale=1 1 1; visual mesh filename=meshes/Right_Gripper.stl scale=1 1 1
- link right_s2: geometry collision mesh filename=meshes/Right_S2.stl scale=1 1 1; visual mesh filename=meshes/Right_S2.stl scale=1 1 1
- link right_s3: geometry collision mesh filename=meshes/Right_S3.stl scale=1 1 1; visual mesh filename=meshes/Right_S3.stl scale=1 1 1
- link right_w0: geometry collision mesh filename=meshes/Right_W0.stl scale=1 1 1; visual mesh filename=meshes/Right_W0.stl scale=1 1 1
- link right_w1: geometry collision mesh filename=meshes/Right_W1.stl scale=1 1 1; visual mesh filename=meshes/Right_W1.stl scale=1 1 1
- link right_w2: geometry collision mesh filename=meshes/Right_W2.stl scale=1 1 1; visual mesh filename=meshes/Right_W2.stl scale=1 1 1
- link s1: geometry collision mesh filename=meshes/S1.stl scale=1 1 1; visual mesh filename=meshes/S1.stl scale=1 1 1
Joints:
- joint __split_right_arm_base_to_original_root: origin xyz=0.85999999999999999 0 0.12999999999999975 rpy=1.5707963267948963 0 -1.5707963267948966 -> xyz=-0.85999999999999999 0 -0.12999999999999975 rpy=-1.570796326794897 0 -1.5707963267948966

Commit message: testing urdf-split final version and urdf validator

File: src/robot/urdf/axol-left.urdf (robot description, URDF)
Before this commit: robot assembly, 20 links, 19 joints
Links:
- link base: geometry collision mesh filename=/home/reforge/Desktop/almond/reforge-interface/src/robot/ur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 scale=1 1 1; visual mesh filename=/home/reforge/Desktop/almond/reforge-interface/src/robot/ur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 scale=1 1 1
- link left_e1: geometry collision mesh filename=/home/reforge/Desktop/almond/reforge-interface/src/robot/ur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 scale=1 1 1; visual mesh filename=/home/reforge/Desktop/almond/reforge-interface/src/robot/ur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 scale=1 1 1
- link left_e2: geometry collision mesh filename=/home/reforge/Desktop/almond/reforge-interface/src/robot/ur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 scale=1 1 1; visual mesh filename=/home/reforge/Desktop/almond/reforge-interface/src/robot/ur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 scale=1 1 1
- link left_gripper: geometry collision mesh filename=/home/reforge/Desktop/almond/reforge-interface/src/robot/ur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 scale=1 1 1; visual mesh filename=/home/reforge/Desktop/almond/reforge-interface/src/robot/ur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 scale=1 1 1
- link left_s2: geometry collision mesh filename=/home/reforge/Desktop/almond/reforge-interface/src/robot/ur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 scale=1 1 1; visual mesh filename=/home/reforge/Desktop/almond/reforge-interface/src/robot/ur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 scale=1 1 1
- link left_s3: geometry collision mesh filename=/home/reforge/Desktop/almond/reforge-interface/src/robot/ur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 scale=1 1 1; visual mesh filename=/home/reforge/Desktop/almond/reforge-interface/src/robot/ur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 scale=1 1 1
- link left_w0: geometry collision mesh filename=/home/reforge/Desktop/almond/reforge-interface/src/robot/ur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 scale=1 1 1; visual mesh filename=/home/reforge/Desktop/almond/reforge-interface/src/robot/ur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 scale=1 1 1
- link left_w1: geometry collision mesh filename=/home/reforge/Desktop/almond/reforge-interface/src/robot/ur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 scale=1 1 1; visual mesh filename=/home/reforge/Desktop/almond/reforge-interface/src/robot/ur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 scale=1 1 1
- link left_w2: geometry collision mesh filename=/home/reforge/Desktop/almond/reforge-interface/src/robot/ur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 scale=1 1 1; visual mesh filename=/home/reforge/Desktop/almond/reforge-interface/src/robot/ur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 scale=1 1 1
- link right_e1: geometry collision mesh filename=/home/reforge/Desktop/almond/reforge-interface/src/robot/ur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 scale=1 1 1; visual mesh filename=/home/reforge/Desktop/almond/reforge-interface/src/robot/ur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 scale=1 1 1
- link right_e2: geometry collision mesh filename=/home/reforge/Desktop/almond/reforge-interface/src/robot/ur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 scale=1 1 1; visual mesh filename=/home/reforge/Desktop/almond/reforge-interface/src/robot/ur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 scale=1 1 1
- link right_gripper: geometry collision mesh filename=/home/reforge/Desktop/almond/reforge-interface/src/robot/ur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 scale=1 1 1; visual mesh filename=/home/reforge/Desktop/almond/reforge-interface/src/robot/ur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 scale=1 1 1
- link right_s2: geometry collision mesh filename=/home/reforge/Desktop/almond/reforge-interface/src/robot/ur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 scale=1 1 1; visual mesh filename=/home/reforge/Desktop/almond/reforge-interface/src/robot/ur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 scale=1 1 1
- link right_s3: geometry collision mesh filename=/home/reforge/Desktop/almond/reforge-interface/src/robot/ur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 scale=1 1 1; visual mesh filename=/home/reforge/Desktop/almond/reforge-interface/src/robot/ur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 scale=1 1 1
- link right_w0: geometry collision mesh filename=/home/reforge/Desktop/almond/reforge-interface/src/robot/ur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 scale=1 1 1; visual mesh filename=/home/reforge/Desktop/almond/reforge-interface/src/robot/ur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 scale=1 1 1
- link right_w1: geometry collision mesh filename=/home/reforge/Desktop/almond/reforge-interface/src/robot/ur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 scale=1 1 1; visual mesh filename=/home/reforge/Desktop/almond/reforge-interface/src/robot/ur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 scale=1 1 1
- link right_w2: geometry collision mesh filename=/home/reforge/Desktop/almond/reforge-interface/src/robot/ur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 scale=1 1 1; visual mesh filename=/home/reforge/Desktop/almond/reforge-interface/src/robot/ur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 scale=1 1 1
- link s1: geometry collision mesh filename=/home/reforge/Desktop/almond/reforge-interface/src/robot/ur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 scale=1 1 1; visual mesh filename=/home/reforge/Desktop/almond/reforge-interface/src/robot/ur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 scale=1 1 1

File: src/robot/urdf/axol-right.urdf (robot description, URDF)
Before this commit: robot assembly, 20 links, 19 joints
Links:
- link base: geometry collision mesh filename=/home/reforge/Desktop/almond/reforge-interface/src/robot/ur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 scale=1 1 1; visual mesh filename=/home/reforge/Desktop/almond/reforge-interface/src/robot/ur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 scale=1 1 1
- link left_e1: geometry collision mesh filename=/home/reforge/Desktop/almond/reforge-interface/src/robot/ur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 scale=1 1 1; visual mesh filename=/home/reforge/Desktop/almond/reforge-interface/src/robot/ur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 scale=1 1 1
- link left_e2: geometry collision mesh filename=/home/reforge/Desktop/almond/reforge-interface/src/robot/ur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 scale=1 1 1; visual mesh filename=/home/reforge/Desktop/almond/reforge-interface/src/robot/ur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 scale=1 1 1
- link left_gripper: geometry collision mesh filename=/home/reforge/Desktop/almond/reforge-interface/src/robot/ur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 scale=1 1 1; visual mesh filename=/home/reforge/Desktop/almond/reforge-interface/src/robot/ur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 scale=1 1 1
- link left_s2: geometry collision mesh filename=/home/reforge/Desktop/almond/reforge-interface/src/robot/ur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 scale=1 1 1; visual mesh filename=/home/reforge/Desktop/almond/reforge-interface/src/robot/ur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 scale=1 1 1
- link left_s3: geometry collision mesh filename=/home/reforge/Desktop/almond/reforge-interface/src/robot/ur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 scale=1 1 1; visual mesh filename=/home/reforge/Desktop/almond/reforge-interface/src/robot/ur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 scale=1 1 1
- link left_w0: geometry collision mesh filename=/home/reforge/Desktop/almond/reforge-interface/src/robot/ur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 scale=1 1 1; visual mesh filename=/home/reforge/Desktop/almond/reforge-interface/src/robot/ur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 scale=1 1 1
- link left_w1: geometry collision mesh filename=/home/reforge/Desktop/almond/reforge-interface/src/robot/ur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 scale=1 1 1; visual mesh filename=/home/reforge/Desktop/almond/reforge-interface/src/robot/ur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 scale=1 1 1
- link left_w2: geometry collision mesh filename=/home/reforge/Desktop/almond/reforge-interface/src/robot/ur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 scale=1 1 1; visual mesh filename=/home/reforge/Desktop/almond/reforge-interface/src/robot/ur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 scale=1 1 1
- link right_e1: geometry collision mesh filename=/home/reforge/Desktop/almond/reforge-interface/src/robot/ur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 scale=1 1 1; visual mesh filename=/home/reforge/Desktop/almond/reforge-interface/src/robot/ur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 scale=1 1 1
- link right_e2: geometry collision mesh filename=/home/reforge/Desktop/almond/reforge-interface/src/robot/ur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 scale=1 1 1; visual mesh filename=/home/reforge/Desktop/almond/reforge-interface/src/robot/ur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 scale=1 1 1
- link right_gripper: geometry collision mesh filename=/home/reforge/Desktop/almond/reforge-interface/src/robot/ur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 scale=1 1 1; visual mesh filename=/home/reforge/Desktop/almond/reforge-interface/src/robot/ur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 scale=1 1 1
- link right_s2: geometry collision mesh filename=/home/reforge/Desktop/almond/reforge-interface/src/robot/ur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 scale=1 1 1; visual mesh filename=/home/reforge/Desktop/almond/reforge-interface/src/robot/ur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 scale=1 1 1
- link right_s3: geometry collision mesh filename=/home/reforge/Desktop/almond/reforge-interface/src/robot/ur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 scale=1 1 1; visual mesh filename=/home/reforge/Desktop/almond/reforge-interface/src/robot/ur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 scale=1 1 1
- link right_w0: geometry collision mesh filename=/home/reforge/Desktop/almond/reforge-interface/src/robot/ur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 scale=1 1 1; visual mesh filename=/home/reforge/Desktop/almond/reforge-interface/src/robot/ur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 scale=1 1 1
- link right_w1: geometry collision mesh filename=/home/reforge/Desktop/almond/reforge-interface/src/robot/ur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 scale=1 1 1; visual mesh filename=/home/reforge/Desktop/almond/reforge-interface/src/robot/ur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 scale=1 1 1
- link right_w2: geometry collision mesh filename=/home/reforge/Desktop/almond/reforge-interface/src/robot/ur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 scale=1 1 1; visual mesh filename=/home/reforge/Desktop/almond/reforge-interface/src/robot/ur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 scale=1 1 1
- link s1: geometry collision mesh filename=/home/reforge/Desktop/almond/reforge-interface/src/robot/ur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 scale=1 1 1; visual mesh filename=/home/reforge/Desktop/almond/reforge-interface/src/robot/ur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 scale=1 1 1
